File: KiCad Projects/Pico 2 C/Pico 2 C.kicad_pcb (KiCad board)
At the start: 2 copper layers, 53.7 x 21 mm, 67 parts, among them J3 USB_C_Receptacle_USB2.0_16P, J4 SM03B-SRSS-TB, Q1 DMG1012T-7, SW1 PTS810 SJK 250 SMTR LFS, U1 RP2350_60QFN, U2 RT6150B-33GQW, U3 W25Q32RVXHJQ TR, Y1 ECS-120-8-33-JGN-TR

Commit message: Replace Inductor
Replaces the stand-in 0602 inductor with the one given in the RP2350 datasheet (AOTA-B201610S3R3-101-T).
Parts:
- L2: footprint Inductor_SMD:L_0603_1608Metric -> Pico 2 C:AOTA-B201610S3R3-101-T
- moved L2 0.11 mm to (157.1, 106.6)
Routing:
- net +1V1: track 19.6 -> 20.3 mm
