File: KiCad Projects/Pico 2 C/RP2350.kicad_sch (KiCad schematic)
At the start: 24 parts, among them U1 RP2350_60QFN

Commit message: Replace Inductor
Replaces the stand-in 0602 inductor with the one given in the RP2350 datasheet (AOTA-B201610S3R3-101-T).
Parts:
- L2: footprint Inductor_SMD:L_0603_1608Metric -> Pico 2 C:AOTA-B201610S3R3-101-T; symbol Device:L_Small -> Pico 2 C:AOTA-B201610S3R3-101-T
Changed lines of the file:
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@@
+	(wire
+		(pts
+			(xy 152.4 38.1) (xy 152.4 66.04)
+		)
+		(stroke
+			(width 0)
+			(type default)
+		)
+	)
 	(wire
 		(pts
@@
 	(wire
 		(pts
-			(xy 157.48 66.04) (xy 157.48 48.26)
-		)
-		(stroke
-			(width 0)
-			(type default)
-		)
-	)
-	(wire
-		(pts
 			(xy 205.74 71.12) (xy 205.74 73.66)
 		)
@@
 	(wire
 		(pts
-			(xy 152.4 66.04) (xy 152.4 38.1)
-		)
-		(stroke
-			(width 0)
-			(type default)
-		)
-	)
-	(wire
-		(pts
 			(xy 99.06 111.76) (xy 107.95 111.76)
 		)
@@
 		(pts
 			(xy 154.94 142.24) (xy 154.94 134.62)
+		)
+		(stroke
+			(width 0)
+			(type default)
+		)
+	)
+	(wire
+		(pts
+			(xy 157.48 48.26) (xy 157.48 66.04)
 		)
 		(stroke
@@
 	)
 	(symbol
-		(lib_id "Device:L_Small")
+		(lib_id "Pico 2 C:AOTA-B201610S3R3-101-T")
 		(at 154.94 57.15 0)
 		(unit 1)
@@
 			)
 		)
-		(property "Footprint" "Inductor_SMD:L_0603_1608Metric"
+		(property "Footprint" "Pico 2 C:AOTA-B201610S3R3-101-T"
 			(at 154.94 57.15 0)
 			(effects
@@
 			)
 		)
-		(property "Datasheet" "~"
+		(property "Datasheet" "https://www.lcsc.com/datasheet/lcsc_datasheet_2412101620_Abracon-LLC-AOTA-B201610S3R3-101-T_C42411119.pdf"
 			(at 154.94 57.15 0)
 			(effects
